Commit message: Gazebo tags included in URDF for material

File: ros2_ws/src/robot_description/urdf/robot.urdf (robot description, URDF)
Before this commit: robot robot, 4 links, 3 joints
Links:
- removed link link_castor_wheel
- added link link_caster_wheel, mass 1; collision sphere radius=0.10; collision sphere radius=0.2
- link link_chassis: geometry collision mesh filename=package://robot_description/meshes/chassis.stl; visual mesh filename=package://robot_description/meshes/chassis.stl
- link link_right_wheel: geometry collision cylinder length=0.12 radius=0.08; collision cylinder length=0.12 radius=0.4
Joints:
- removed joint joint_chassis_castor_wheel
- added joint joint_chassis_caster_wheel: type fixed, parent link_chassis, child link_caster_wheel, origin xyz=0.8 0 -0.15 rpy=0 0 0
