Commit message: Added ros+gazebo_bridge to launch file

File: ros2_ws/src/robot_description/urdf/robot.xacro (robot description, xacro)
@@ -5,5 +5,5 @@
     <xacro:property name="chassis_mass" value="10" />
     <!-- pi is already defined as a global varibale -->
-    <xacro:property name="pi" value="3.141592654" />
+    <!-- <xacro:property name="pi" value="3.141592654" /> -->
     <!-- Link - chassis -->
     <link name="link_chassis">
